File: usb-c/pcb/usb-c-expansion-card/usb-c-expansion-card.kicad_pcb (KiCad board)
At the start: 4 copper layers, 26 x 30 mm, 15 parts, among them J1 USB_C_Receptacle, P1 USB_C_Plug, U1 USBLC6-2SC6, U2 USBLC6-2SC6, U3 USBLC6-2SC6

Commit message: changes on chassis, accommodating for PCB
Signed-off-by: Lucy <user@domain.tld>
Parts:
- moved P1 1.29 mm to (140.0, 130.3)
Routing:
- net /VBUS: track 54.5 -> 51.9 mm
- net /OUT_D_P: track 16.2 -> 14.9 mm
- net /VCONN: track 17.6 -> 16.3 mm
- net /ESD_RX2_N: track 24.4 -> 23.1 mm
- net /ESD_TX1_N: track 24.9 -> 23.6 mm
- net /ESD_TX1_P: track 25.0 -> 23.7 mm
- net /ESD_RX1_N: track 28.5 -> 27.2 mm
- net /CC: track 11.4 -> 10.1 mm
- net /OUT_SBU2: track 11.7 -> 10.4 mm
- net /OUT_SBU1: track 11.9 -> 10.6 mm
- net /ESD_RX1_P: track 28.6 -> 27.3 mm
- net /OUT_D_N: track 16.2 -> 15.0 mm
- net /ESD_RX2_P: track 24.5 -> 23.3 mm
- net GND: vias 62 -> 47
Other:
- board size 26 x 30 mm -> 26 x 28.7 mm
